Commit message: imu-test

File: digital-twin-service/go1-base/catkin_ws/src/qre_go1/go1_description/urdf/go1.urdf (robot description, URDF)
Before this commit: robot go1, 38 links, 37 joints
Links:
- added link laser_link, mass 1e-5; collision cylinder length=0.05 radius=0.05; visual cylinder length=0.05 radius=0.05
- added link phidgets_imu_link, mass 0.001; collision box size=0.001 0.001 0.001; visual box size=0.001 0.001 0.001
Joints:
- added joint laser_joint: type fixed, parent trunk, child laser_link, origin xyz=0.05 0 0.08 rpy=0 0 0
- added joint phidgets_imu_joint: type fixed, parent base, child phidgets_imu_link, origin xyz=0 0 0 rpy=0 0 0
- joint FL_calf_joint: limit lower=-2.72271363311 upper=-0.837758040957 effort=23.7 velocity=30.1 -> lower=-2.722713633111154 upper=-0.8377580409572781 effort=23.7 velocity=30.1
- joint FL_hip_joint: limit lower=-1.0471975512 upper=1.0471975512 effort=23.7 velocity=30.1 -> lower=-1.0471975511965976 upper=1.0471975511965976 effort=23.7 velocity=30.1
- joint FL_thigh_joint: limit lower=-0.663225115758 upper=2.96705972839 effort=23.7 velocity=30.1 -> lower=-0.6632251157578452 upper=2.9670597283903604 effort=23.7 velocity=30.1
- joint FR_calf_joint: limit lower=-2.72271363311 upper=-0.837758040957 effort=23.7 velocity=30.1 -> lower=-2.722713633111154 upper=-0.8377580409572781 effort=23.7 velocity=30.1
- joint FR_hip_joint: limit lower=-1.0471975512 upper=1.0471975512 effort=23.7 velocity=30.1 -> lower=-1.0471975511965976 upper=1.0471975511965976 effort=23.7 velocity=30.1
- joint FR_thigh_joint: limit lower=-0.663225115758 upper=2.96705972839 effort=23.7 velocity=30.1 -> lower=-0.6632251157578452 upper=2.9670597283903604 effort=23.7 velocity=30.1
- joint RL_calf_joint: limit lower=-2.72271363311 upper=-0.837758040957 effort=23.7 velocity=30.1 -> lower=-2.722713633111154 upper=-0.8377580409572781 effort=23.7 velocity=30.1
- joint RL_hip_joint: limit lower=-1.0471975512 upper=1.0471975512 effort=23.7 velocity=30.1 -> lower=-1.0471975511965976 upper=1.0471975511965976 effort=23.7 velocity=30.1
- joint RL_thigh_joint: limit lower=-0.663225115758 upper=2.96705972839 effort=23.7 velocity=30.1 -> lower=-0.6632251157578452 upper=2.9670597283903604 effort=23.7 velocity=30.1
- joint RR_calf_joint: limit lower=-2.72271363311 upper=-0.837758040957 effort=23.7 velocity=30.1 -> lower=-2.722713633111154 upper=-0.8377580409572781 effort=23.7 velocity=30.1
- joint RR_hip_joint: limit lower=-1.0471975512 upper=1.0471975512 effort=23.7 velocity=30.1 -> lower=-1.0471975511965976 upper=1.0471975511965976 effort=23.7 velocity=30.1
- joint RR_thigh_joint: limit lower=-0.663225115758 upper=2.96705972839 effort=23.7 velocity=30.1 -> lower=-0.6632251157578452 upper=2.9670597283903604 effort=23.7 velocity=30.1
- joint camera_joint_chin: origin xyz=0.2522 0.0125 -0.0436 rpy=3.14159265359 1.57079632679 0 -> xyz=0.2522 0.0125 -0.0436 rpy=3.141592653589793 1.5707963267948966 0
- joint camera_joint_face: origin xyz=0.2785 0.0125 0.0167 rpy=3.14159265359 0 0 -> xyz=0.2785 0.0125 0.0167 rpy=3.141592653589793 0 0
- joint camera_joint_left: origin xyz=-0.066 0.082 -0.0176 rpy=3.14159265359 0.2618 1.57079632679 -> xyz=-0.066 0.082 -0.0176 rpy=3.141592653589793 0.2618 1.5707963267948966
- joint camera_joint_rearDown: origin xyz=-0.0825 0.0125 -0.04365 rpy=3.14159265359 1.57079632679 0 -> xyz=-0.0825 0.0125 -0.04365 rpy=3.141592653589793 1.5707963267948966 0
- joint camera_joint_right: origin xyz=-0.041 -0.082 -0.0176 rpy=3.14159265359 0.2618 -1.57079632679 -> xyz=-0.041 -0.082 -0.0176 rpy=3.141592653589793 0.2618 -1.5707963267948966
- joint camera_optical_joint_chin: origin xyz=0 0 0 rpy=-1.57079632679 0 -1.57079632679 -> xyz=0 0 0 rpy=-1.5707963267948966 0 -1.5707963267948966
- joint camera_optical_joint_face: origin xyz=0 0 0 rpy=-1.57079632679 0 -1.57079632679 -> xyz=0 0 0 rpy=-1.5707963267948966 0 -1.5707963267948966
- joint camera_optical_joint_left: origin xyz=0 0 0 rpy=-1.57079632679 0 -1.57079632679 -> xyz=0 0 0 rpy=-1.5707963267948966 0 -1.5707963267948966
- joint camera_optical_joint_rearDown: origin xyz=0 0 0 rpy=-1.57079632679 0 -1.57079632679 -> xyz=0 0 0 rpy=-1.5707963267948966 0 -1.5707963267948966
- joint camera_optical_joint_right: origin xyz=0 0 0 rpy=-1.57079632679 0 -1.57079632679 -> xyz=0 0 0 rpy=-1.5707963267948966 0 -1.5707963267948966
- joint ultraSound_joint_left: origin xyz=-0.0535  0.0826 0.00868 rpy=0 0.2618 1.57079632679 -> xyz=-0.0535  0.0826 0.00868 rpy=0 0.2618 1.5707963267948966
- joint ultraSound_joint_right: origin xyz=-0.0535 -0.0826 0.00868 rpy=0 0.2618 -1.57079632679 -> xyz=-0.0535 -0.0826 0.00868 rpy=0 0.2618 -1.5707963267948966

File: digital-twin-service/go1-base/catkin_ws/src/qre_go1/go1_description/xacro/robot.xacro (robot description, xacro)
@@ -30,4 +30,25 @@
             </geometry>
         </visual>
+    </link>
+    <!-- Phidgets IMU mounted to the base frame -->
+    <joint name="phidgets_imu_joint" type="fixed">
+        <parent link="base"/>
+        <child link="phidgets_imu_link"/>
+        <!-- Set these to the IMU’s position/orientation relative to base -->
+        <origin xyz="0 0 0" rpy="0 0 0"/>
+    </joint>
+    <link name="phidgets_imu_link">
+        <inertial>
+            <mass value="0.001"/>
+            <origin xyz="0 0 0" rpy="0 0 0"/>
+            <inertia ixx="1e-4" ixy="0" ixz="0" iyy="1e-4" iyz="0" izz="1e-4"/>
+        </inertial>
+        <visual>
+            <geometry><box size="0.001 0.001 0.001"/></geometry>
+            <material name="black"/>
+        </visual>
+        <collision>
+            <geometry><box size="0.001 0.001 0.001"/></geometry>
+        </collision>
     </link>
     <joint name="floating_base" type="fixed">

Commit message: final-test

File: digital-twin-service/go1-base/catkin_ws/src/qre_go1/go1_description/urdf/go1.urdf (robot description, URDF)
Before this commit: robot go1, 40 links, 39 joints
Links:
- removed link FL_thigh_shoulder
- removed link FR_thigh_shoulder
- removed link RL_thigh_shoulder
- removed link RR_thigh_shoulder
- removed link laser_link
- removed link phidgets_imu_link
- added link FL_calf_rotor, mass 0.089; collision cylinder length=0.02 radius=0.035; visual cylinder length=0.02 radius=0.035
- added link FL_hip_rotor, mass 0.089; collision cylinder length=0.02 radius=0.035; visual cylinder length=0.02 radius=0.035
- added link FL_thigh_rotor, mass 0.089; collision cylinder length=0.02 radius=0.035; visual cylinder length=0.02 radius=0.035
- added link FR_calf_rotor, mass 0.089; collision cylinder length=0.02 radius=0.035; visual cylinder length=0.02 radius=0.035
- added link FR_hip_rotor, mass 0.089; collision cylinder length=0.02 radius=0.035; visual cylinder length=0.02 radius=0.035
- added link FR_thigh_rotor, mass 0.089; collision cylinder length=0.02 radius=0.035; visual cylinder length=0.02 radius=0.035
- added link RL_calf_rotor, mass 0.089; collision cylinder length=0.02 radius=0.035; visual cylinder length=0.02 radius=0.035
- added link RL_hip_rotor, mass 0.089; collision cylinder length=0.02 radius=0.035; visual cylinder length=0.02 radius=0.035
- added link RL_thigh_rotor, mass 0.089; collision cylinder length=0.02 radius=0.035; visual cylinder length=0.02 radius=0.035
- added link RR_calf_rotor, mass 0.089; collision cylinder length=0.02 radius=0.035; visual cylinder length=0.02 radius=0.035
- added link RR_hip_rotor, mass 0.089; collision cylinder length=0.02 radius=0.035; visual cylinder length=0.02 radius=0.035
- added link RR_thigh_rotor, mass 0.089; collision cylinder length=0.02 radius=0.035; visual cylinder length=0.02 radius=0.035
- link FL_calf: mass 0.131 -> 0.135862
- link FR_calf: mass 0.131 -> 0.135862
- link RL_calf: mass 0.131 -> 0.135862
- link RR_calf: mass 0.131 -> 0.135862
Joints:
- removed joint FL_hip_fixed
- removed joint FR_hip_fixed
- removed joint RL_hip_fixed
- removed joint RR_hip_fixed
- removed joint laser_joint
- removed joint phidgets_imu_joint
- added joint FL_calf_rotor_joint: type fixed, parent FL_thigh, child FL_calf_rotor, origin xyz=0.0 -0.03235 0 rpy=0 0 0
- added joint FL_hip_rotor_joint: type fixed, parent trunk, child FL_hip_rotor, origin xyz=0.11215 0.04675 0 rpy=0 0 0
- added joint FL_thigh_rotor_joint: type fixed, parent FL_hip, child FL_thigh_rotor, origin xyz=0.0 -0.00015 0 rpy=0 0 0
- added joint FR_calf_rotor_joint: type fixed, parent FR_thigh, child FR_calf_rotor, origin xyz=0.0 0.03235 0 rpy=0 0 0
- added joint FR_hip_rotor_joint: type fixed, parent trunk, child FR_hip_rotor, origin xyz=0.11215 -0.04675 0 rpy=0 0 0
- added joint FR_thigh_rotor_joint: type fixed, parent FR_hip, child FR_thigh_rotor, origin xyz=0.0 0.00015 0 rpy=0 0 0
- added joint RL_calf_rotor_joint: type fixed, parent RL_thigh, child RL_calf_rotor, origin xyz=0.0 -0.03235 0 rpy=0 0 0
- added joint RL_hip_rotor_joint: type fixed, parent trunk, child RL_hip_rotor, origin xyz=-0.11215 0.04675 0 rpy=0 0 0
- added joint RL_thigh_rotor_joint: type fixed, parent RL_hip, child RL_thigh_rotor, origin xyz=0.0 -0.00015 0 rpy=0 0 0
- added joint RR_calf_rotor_joint: type fixed, parent RR_thigh, child RR_calf_rotor, origin xyz=0.0 0.03235 0 rpy=0 0 0
- added joint RR_hip_rotor_joint: type fixed, parent trunk, child RR_hip_rotor, origin xyz=-0.11215 -0.04675 0 rpy=0 0 0
- added joint RR_thigh_rotor_joint: type fixed, parent RR_hip, child RR_thigh_rotor, origin xyz=0.0 0.00015 0 rpy=0 0 0
- joint FL_calf_joint: limit lower=-2.722713633111154 upper=-0.8377580409572781 effort=23.7 velocity=30.1 -> lower=-2.818 upper=-0.888 effort=35.55 velocity=20.06
- joint FL_hip_joint: limit lower=-1.0471975511965976 upper=1.0471975511965976 effort=23.7 velocity=30.1 -> lower=-0.863 upper=0.863 effort=23.7 velocity=30.1
- joint FL_thigh_joint: limit lower=-0.6632251157578452 upper=2.9670597283903604 effort=23.7 velocity=30.1 -> lower=-0.686 upper=4.501 effort=23.7 velocity=30.1
- joint FR_calf_joint: limit lower=-2.722713633111154 upper=-0.8377580409572781 effort=23.7 velocity=30.1 -> lower=-2.818 upper=-0.888 effort=35.55 velocity=20.06
- joint FR_hip_joint: limit lower=-1.0471975511965976 upper=1.0471975511965976 effort=23.7 velocity=30.1 -> lower=-0.863 upper=0.863 effort=23.7 velocity=30.1
- joint FR_thigh_joint: limit lower=-0.6632251157578452 upper=2.9670597283903604 effort=23.7 velocity=30.1 -> lower=-0.686 upper=4.501 effort=23.7 velocity=30.1
- joint RL_calf_joint: limit lower=-2.722713633111154 upper=-0.8377580409572781 effort=23.7 velocity=30.1 -> lower=-2.818 upper=-0.888 effort=35.55 velocity=20.06
- joint RL_hip_joint: limit lower=-1.0471975511965976 upper=1.0471975511965976 effort=23.7 velocity=30.1 -> lower=-0.863 upper=0.863 effort=23.7 velocity=30.1
- joint RL_thigh_joint: limit lower=-0.6632251157578452 upper=2.9670597283903604 effort=23.7 velocity=30.1 -> lower=-0.686 upper=4.501 effort=23.7 velocity=30.1
- joint RR_calf_joint: limit lower=-2.722713633111154 upper=-0.8377580409572781 effort=23.7 velocity=30.1 -> lower=-2.818 upper=-0.888 effort=35.55 velocity=20.06
- joint RR_hip_joint: limit lower=-1.0471975511965976 upper=1.0471975511965976 effort=23.7 velocity=30.1 -> lower=-0.863 upper=0.863 effort=23.7 velocity=30.1
- joint RR_thigh_joint: limit lower=-0.6632251157578452 upper=2.9670597283903604 effort=23.7 velocity=30.1 -> lower=-0.686 upper=4.501 effort=23.7 velocity=30.1

File: digital-twin-service/go1-base/catkin_ws/src/qre_go1/go1_description/xacro/robot.xacro (robot description, xacro)
@@ -10,8 +10,7 @@
     <xacro:include filename="$(find go1_description)/xacro/ultraSound.xacro"/>
     <!-- <xacro:include filename="$(find go1_gazebo)/launch/stairs.urdf.xacro"/> -->
-    <xacro:include filename="$(find go1_description)/xacro/lidar.xacro"/>
     <!-- <xacro:stairs stairs="15" xpos="0" ypos="0" zpos="0" /> -->
-    <!-- Rollover Protection mode will add an additional stick on the top, use "true" or "false" to switch it. -->
-    <xacro:property name="rolloverProtection" value="false"/>
+    <!-- Rotor related joint and link is only for demonstrate location. -->
+    <!-- Actually, the rotor will rotate and the joint is not fixed. Reduction ratio should be considered. -->
     <!-- Debug mode will hung up the robot, use "true" or "false" to switch it. -->
     <xacro:if value="$(arg DEBUG)">
@@ -30,25 +29,4 @@
             </geometry>
         </visual>
-    </link>
-    <!-- Phidgets IMU mounted to the base frame -->
-    <joint name="phidgets_imu_joint" type="fixed">
-        <parent link="base"/>
-        <child link="phidgets_imu_link"/>
-        <!-- Set these to the IMU’s position/orientation relative to base -->
-        <origin xyz="0 0 0" rpy="0 0 0"/>
-    </joint>
-    <link name="phidgets_imu_link">
-        <inertial>
-            <mass value="0.001"/>
-            <origin xyz="0 0 0" rpy="0 0 0"/>
-            <inertia ixx="1e-4" ixy="0" ixz="0" iyy="1e-4" iyz="0" izz="1e-4"/>
-        </inertial>
-        <visual>
-            <geometry><box size="0.001 0.001 0.001"/></geometry>
-            <material name="black"/>
-        </visual>
-        <collision>
-            <geometry><box size="0.001 0.001 0.001"/></geometry>
-        </collision>
     </link>
     <joint name="floating_base" type="fixed">
@@ -80,33 +58,4 @@
         </inertial>
     </link>
-    <xacro:if value="${(rolloverProtection == 'true')}">
-        <joint name="stick_joint" type="fixed">
-            <parent link="trunk"/>
-            <child link="stick_link"/>
-            <origin rpy="0 0 0" xyz="${0.18} 0 ${stick_length/2.0+0.08}"/>
-        </joint>
-        <link name="stick_link">
-            <visual>
-                <geometry>
-                    <cylinder length="${stick_length}" radius="${stick_radius}"/>
-                </geometry>
-                <origin rpy="0 0 0" xyz="0 0 0"/>
-                <!-- <material name="white"/> -->
-            </visual>
-            <collision>
-                <geometry>
-                    <cylinder length="${stick_length}" radius="${stick_radius}"/>
-                </geometry>
-                <origin rpy="0 0 0" xyz="0 0 0"/>
-            </collision>
-            <inertial>
-                <mass value="${stick_mass}"/>
-                <inertia
-                    ixx="${stick_mass / 2.0 * (stick_radius*stick_radius)}" ixy="0.0" ixz="0.0"
-                    iyy="${stick_mass / 12.0 * (3*stick_radius*stick_radius + stick_length*stick_length)}" iyz="0.0"
-                    izz="${stick_mass / 12.0 * (3*stick_radius*stick_radius + stick_length*stick_length)}"/>
-            </inertial>
-        </link>
-    </xacro:if>
     <joint name="imu_joint" type="fixed">
         <parent link="trunk"/>
@@ -134,16 +83,8 @@
         </collision>
     </link>
-    <xacro:leg name="FR" mirror="-1" mirror_dae="False" front_hind="1" front_hind_dae="True">
-        <origin rpy="0 0 0" xyz="${leg_offset_x} ${-leg_offset_y} 0"/>
-    </xacro:leg>
-    <xacro:leg name="FL" mirror="1" mirror_dae="True" front_hind="1" front_hind_dae="True">
-        <origin rpy="0 0 0" xyz="${leg_offset_x} ${leg_offset_y} 0"/>
-    </xacro:leg>
-    <xacro:leg name="RR" mirror="-1" mirror_dae="False" front_hind="-1" front_hind_dae="False">
-        <origin rpy="0 0 0" xyz="${-leg_offset_x} ${-leg_offset_y} 0"/>
-    </xacro:leg>
-    <xacro:leg name="RL" mirror="1" mirror_dae="True" front_hind="-1" front_hind_dae="False">
-        <origin rpy="0 0 0" xyz="${-leg_offset_x} ${leg_offset_y} 0"/>
-    </xacro:leg>
+    <xacro:leg name="FR" mirror="-1" mirror_dae= "False" front_hind="1"  front_hind_dae="True"  />
+    <xacro:leg name="FL" mirror="1"  mirror_dae="True"   front_hind="1"  front_hind_dae="True"  />
+    <xacro:leg name="RR" mirror="-1" mirror_dae="False"  front_hind="-1" front_hind_dae="False" />
+    <xacro:leg name="RL" mirror="1"  mirror_dae="True"   front_hind="-1" front_hind_dae="False" />
     <xacro:depthCamera camID="1" name="face">
         <origin rpy="${PI} 0 0" xyz="0.2785 0.0125 0.0167"/>
@@ -184,6 +125,3 @@
         <origin rpy="0 0 0" xyz="0.2747 0.0 -0.0088"/>
     </xacro:ultraSound>
-    <xacro:lidar parent="trunk">
-        <origin rpy="0 0 0" xyz="0.05 0 0.08"/>
-    </xacro:lidar>
 </robot>
