Commit message: c

File: digital-twin-service/go1-base/catkin_ws/src/qre_go1/go1_description/urdf/go1.urdf (robot description, URDF)
Before this commit: robot go1, 46 links, 45 joints
Links:
- removed link FL_calf_rotor
- removed link FL_hip_rotor
- removed link FL_thigh_rotor
- removed link FR_calf_rotor
- removed link FR_hip_rotor
- removed link FR_thigh_rotor
- removed link RL_calf_rotor
- removed link RL_hip_rotor
- removed link RL_thigh_rotor
- removed link RR_calf_rotor
- removed link RR_hip_rotor
- removed link RR_thigh_rotor
- added link FL_thigh_shoulder; collision cylinder length=0.032 radius=0.041
- added link FR_thigh_shoulder; collision cylinder length=0.032 radius=0.041
- added link RL_thigh_shoulder; collision cylinder length=0.032 radius=0.041
- added link RR_thigh_shoulder; collision cylinder length=0.032 radius=0.041
- added link laser_link, mass 1e-5; collision cylinder length=0.05 radius=0.05; visual cylinder length=0.05 radius=0.05
- added link phidgets_imu_link, mass 0.001; collision box size=0.001 0.001 0.001; visual box size=0.001 0.001 0.001
- link FL_calf: mass 0.135862 -> 0.131
- link FR_calf: mass 0.135862 -> 0.131
- link RL_calf: mass 0.135862 -> 0.131
- link RR_calf: mass 0.135862 -> 0.131
Joints:
- removed joint FL_calf_rotor_joint
- removed joint FL_hip_rotor_joint
- removed joint FL_thigh_rotor_joint
- removed joint FR_calf_rotor_joint
- removed joint FR_hip_rotor_joint
- removed joint FR_thigh_rotor_joint
- removed joint RL_calf_rotor_joint
- removed joint RL_hip_rotor_joint
- removed joint RL_thigh_rotor_joint
- removed joint RR_calf_rotor_joint
- removed joint RR_hip_rotor_joint
- removed joint RR_thigh_rotor_joint
- added joint FL_hip_fixed: type fixed, parent FL_hip, child FL_thigh_shoulder, origin xyz=0 0.08 0 rpy=0 0 0
- added joint FR_hip_fixed: type fixed, parent FR_hip, child FR_thigh_shoulder, origin xyz=0 -0.08 0 rpy=0 0 0
- added joint RL_hip_fixed: type fixed, parent RL_hip, child RL_thigh_shoulder, origin xyz=0 0.08 0 rpy=0 0 0
- added joint RR_hip_fixed: type fixed, parent RR_hip, child RR_thigh_shoulder, origin xyz=0 -0.08 0 rpy=0 0 0
- added joint laser_joint: type fixed, parent trunk, child laser_link, origin xyz=0.05 0 0.08 rpy=0 0 0
- added joint phidgets_imu_joint: type fixed, parent base, child phidgets_imu_link, origin xyz=0 0 0 rpy=0 0 0
- joint FL_calf_joint: limit lower=-2.818 upper=-0.888 effort=35.55 velocity=20.06 -> lower=-2.722713633111154 upper=-0.8377580409572781 effort=23.7 velocity=30.1
- joint FL_hip_joint: limit lower=-0.863 upper=0.863 effort=23.7 velocity=30.1 -> lower=-1.0471975511965976 upper=1.0471975511965976 effort=23.7 velocity=30.1
- joint FL_thigh_joint: limit lower=-0.686 upper=4.501 effort=23.7 velocity=30.1 -> lower=-0.6632251157578452 upper=2.9670597283903604 effort=23.7 velocity=30.1
- joint FR_calf_joint: limit lower=-2.818 upper=-0.888 effort=35.55 velocity=20.06 -> lower=-2.722713633111154 upper=-0.8377580409572781 effort=23.7 velocity=30.1
- joint FR_hip_joint: limit lower=-0.863 upper=0.863 effort=23.7 velocity=30.1 -> lower=-1.0471975511965976 upper=1.0471975511965976 effort=23.7 velocity=30.1
- joint FR_thigh_joint: limit lower=-0.686 upper=4.501 effort=23.7 velocity=30.1 -> lower=-0.6632251157578452 upper=2.9670597283903604 effort=23.7 velocity=30.1
- joint RL_calf_joint: limit lower=-2.818 upper=-0.888 effort=35.55 velocity=20.06 -> lower=-2.722713633111154 upper=-0.8377580409572781 effort=23.7 velocity=30.1
- joint RL_hip_joint: limit lower=-0.863 upper=0.863 effort=23.7 velocity=30.1 -> lower=-1.0471975511965976 upper=1.0471975511965976 effort=23.7 velocity=30.1
- joint RL_thigh_joint: limit lower=-0.686 upper=4.501 effort=23.7 velocity=30.1 -> lower=-0.6632251157578452 upper=2.9670597283903604 effort=23.7 velocity=30.1
- joint RR_calf_joint: limit lower=-2.818 upper=-0.888 effort=35.55 velocity=20.06 -> lower=-2.722713633111154 upper=-0.8377580409572781 effort=23.7 velocity=30.1
- joint RR_hip_joint: limit lower=-0.863 upper=0.863 effort=23.7 velocity=30.1 -> lower=-1.0471975511965976 upper=1.0471975511965976 effort=23.7 velocity=30.1
- joint RR_thigh_joint: limit lower=-0.686 upper=4.501 effort=23.7 velocity=30.1 -> lower=-0.6632251157578452 upper=2.9670597283903604 effort=23.7 velocity=30.1

File: digital-twin-service/go1-base/catkin_ws/src/qre_go1/go1_description/xacro/const.xacro (robot description, xacro)
@@ -28,38 +28,19 @@
     <!-- <xacro:property name="trunk_offset_z" value="0.01675"/> -->
     <xacro:property name="hip_offset" value="0.08"/>
-    <!-- offset of link and rotor locations (left front) -->
-    <xacro:property name="hip_offset_x" value="0.1881"/>
-    <xacro:property name="hip_offset_y" value="0.04675"/>
-    <xacro:property name="hip_offset_z" value="0.0"/>
-    <xacro:property name="hip_rotor_offset_x" value="0.11215"/>
-    <xacro:property name="hip_rotor_offset_y" value="0.04675"/>
-    <xacro:property name="hip_rotor_offset_z" value="0.0"/>
-    <xacro:property name="thigh_offset_x" value="0"/>
-    <xacro:property name="thigh_offset_y" value="0.08"/>
-    <xacro:property name="thigh_offset_z" value="0.0"/>
-    <xacro:property name="thigh_rotor_offset_x" value="0.0"/>
-    <xacro:property name="thigh_rotor_offset_y" value="-0.00015"/>
-    <xacro:property name="thigh_rotor_offset_z" value="0.0"/>
-    <xacro:property name="calf_offset_x" value="0.0"/>
-    <xacro:property name="calf_offset_y" value="0.0"/>
-    <xacro:property name="calf_offset_z" value="-0.213"/>
-    <xacro:property name="calf_rotor_offset_x" value="0.0"/>
-    <xacro:property name="calf_rotor_offset_y" value="-0.03235"/>
-    <xacro:property name="calf_rotor_offset_z" value="0.0"/>
     <!-- joint limits -->
-    <xacro:property name="damping" value="0.0"/>
-    <xacro:property name="friction" value="0.0"/>
-    <xacro:property name="hip_position_max" value="0.863"/>
-    <xacro:property name="hip_position_min" value="-0.863"/>
+    <xacro:property name="damping" value="0.01"/>
+    <xacro:property name="friction" value="0.2"/>
+    <xacro:property name="hip_max" value="60"/>
+    <xacro:property name="hip_min" value="-60"/>
     <xacro:property name="hip_velocity_max" value="30.1"/>
     <xacro:property name="hip_torque_max" value="23.7"/>
-    <xacro:property name="thigh_position_max" value="4.501"/>
-    <xacro:property name="thigh_position_min" value="-0.686"/>
+    <xacro:property name="thigh_max" value="170"/>
+    <xacro:property name="thigh_min" value="-38"/>
     <xacro:property name="thigh_velocity_max" value="30.1"/>
     <xacro:property name="thigh_torque_max" value="23.7"/>
-    <xacro:property name="calf_position_max" value="-0.888"/>
-    <xacro:property name="calf_position_min" value="-2.818"/>
-    <xacro:property name="calf_velocity_max" value="20.06"/>
-    <xacro:property name="calf_torque_max" value="35.55"/>
+    <xacro:property name="calf_max" value="-48"/>
+    <xacro:property name="calf_min" value="-156"/>
+    <xacro:property name="calf_velocity_max" value="30.1"/>
+    <xacro:property name="calf_torque_max" value="23.7"/>
     <!-- dynamics inertial value        total 12.84kg -->
     <!-- trunk -->
@@ -68,73 +49,43 @@
     <xacro:property name="trunk_com_y" value="0.002"/>
     <xacro:property name="trunk_com_z" value="-0.0005"/>
-    <xacro:property name="trunk_ixx" value="0.0168128557"/>
-    <xacro:property name="trunk_ixy" value="-0.0002296769"/>
-    <xacro:property name="trunk_ixz" value="-0.0002945293"/>
-    <xacro:property name="trunk_iyy" value="0.063009565"/>
-    <xacro:property name="trunk_iyz" value="-0.0000418731"/>
-    <xacro:property name="trunk_izz" value="0.0716547275"/>
+    <xacro:property name="trunk_ixx" value="0.0168352186"/>
+    <xacro:property name="trunk_ixy" value="0.0004636141"/>
+    <xacro:property name="trunk_ixz" value="0.0002367952"/>
+    <xacro:property name="trunk_iyy" value="0.0656071082"/>
+    <xacro:property name="trunk_iyz" value="0.000036671"/>
+    <xacro:property name="trunk_izz" value="0.0742720659"/>
     <!-- hip (left front) -->
     <xacro:property name="hip_mass" value="0.591"/>
-    <xacro:property name="hip_com_x" value="-0.005657"/>
-    <xacro:property name="hip_com_y" value="-0.008752"/>
-    <xacro:property name="hip_com_z" value="-0.000102"/>
-    <xacro:property name="hip_ixx" value="0.000334008405"/>
-    <xacro:property name="hip_ixy" value="-0.000010826066"/>
-    <xacro:property name="hip_ixz" value="0.000001290732"/>
-    <xacro:property name="hip_iyy" value="0.000619101213"/>
-    <xacro:property name="hip_iyz" value="0.000001643194"/>
-    <xacro:property name="hip_izz" value="0.00040057614"/>
-    <xacro:property name="hip_rotor_mass" value="0.089"/>
-    <xacro:property name="hip_rotor_com_x" value="0.0"/>
-    <xacro:property name="hip_rotor_com_y" value="0.0"/>
-    <xacro:property name="hip_rotor_com_z" value="0.0"/>
-    <xacro:property name="hip_rotor_ixx" value="0.000111842"/>
-    <xacro:property name="hip_rotor_ixy" value="0.0"/>
-    <xacro:property name="hip_rotor_ixz" value="0.0"/>
-    <xacro:property name="hip_rotor_iyy" value="0.000059647"/>
-    <xacro:property name="hip_rotor_iyz" value="0.0"/>
-    <xacro:property name="hip_rotor_izz" value="0.000059647"/>
+    <xacro:property name="hip_com_x" value="-0.00541"/>
+    <xacro:property name="hip_com_y" value="-0.00074"/>
+    <xacro:property name="hip_com_z" value="0.000006"/>
+    <xacro:property name="hip_ixx" value="0.000374268192"/>
+    <xacro:property name="hip_ixy" value="0.000036844422"/>
+    <xacro:property name="hip_ixz" value="-0.000000986754"/>
+    <xacro:property name="hip_iyy" value="0.000635923669"/>
+    <xacro:property name="hip_iyz" value="-0.000001172894"/>
+    <xacro:property name="hip_izz" value="0.000457647394"/>
     <!-- thigh -->
     <xacro:property name="thigh_mass" value="0.92"/>
-    <xacro:property name="thigh_com_x" value="-0.003342"/>
-    <xacro:property name="thigh_com_y" value="-0.018054"/>
-    <xacro:property name="thigh_com_z" value="-0.033451"/>
-    <xacro:property name="thigh_ixx" value="0.004431760472"/>
-    <xacro:property name="thigh_ixy" value="0.000057496807"/>
-    <xacro:property name="thigh_ixz" value="-0.000218457134"/>
-    <xacro:property name="thigh_iyy" value="0.004485671726"/>
-    <xacro:property name="thigh_iyz" value="0.000572001265"/>
-    <xacro:property name="thigh_izz" value="0.000740309489"/>
-    <xacro:property name="thigh_rotor_mass" value="0.089"/>
-    <xacro:property name="thigh_rotor_com_x" value="0.0"/>
-    <xacro:property name="thigh_rotor_com_y" value="0.0"/>
-    <xacro:property name="thigh_rotor_com_z" value="0.0"/>
-    <xacro:property name="thigh_rotor_ixx" value="0.000059647"/>
-    <xacro:property name="thigh_rotor_ixy" value="0.0"/>
-    <xacro:property name="thigh_rotor_ixz" value="0.0"/>
-    <xacro:property name="thigh_rotor_iyy" value="0.000111842"/>
-    <xacro:property name="thigh_rotor_iyz" value="0.0"/>
-    <xacro:property name="thigh_rotor_izz" value="0.000059647"/>
+    <xacro:property name="thigh_com_x" value="-0.003468"/>
+    <xacro:property name="thigh_com_y" value="-0.018947"/>
+    <xacro:property name="thigh_com_z" value="-0.032736"/>
+    <xacro:property name="thigh_ixx" value="0.005851561134"/>
+    <xacro:property name="thigh_ixy" value="0.000001783284"/>
+    <xacro:property name="thigh_ixz" value="0.000328291374"/>
+    <xacro:property name="thigh_iyy" value="0.005596155105"/>
+    <xacro:property name="thigh_iyz" value="0.000021430713"/>
+    <xacro:property name="thigh_izz" value="0.00107157026"/>
     <!-- calf -->
-    <xacro:property name="calf_mass" value="0.135862"/>
-    <xacro:property name="calf_com_x" value="0.006197"/>
-    <xacro:property name="calf_com_y" value="0.001408"/>
-    <xacro:property name="calf_com_z" value="-0.116695"/>
-    <xacro:property name="calf_ixx" value="0.001088793059"/>
-    <xacro:property name="calf_ixy" value="-0.000000255679"/>
-    <xacro:property name="calf_ixz" value="0.000007117814"/>
-    <xacro:property name="calf_iyy" value="0.001100428748"/>
-    <xacro:property name="calf_iyz" value="0.000002077264"/>
-    <xacro:property name="calf_izz" value="0.000024787446"/>
-    <xacro:property name="calf_rotor_mass" value="0.089"/>
-    <xacro:property name="calf_rotor_com_x" value="0.0"/>
-    <xacro:property name="calf_rotor_com_y" value="0.0"/>
-    <xacro:property name="calf_rotor_com_z" value="0.0"/>
-    <xacro:property name="calf_rotor_ixx" value="0.000059647"/>
-    <xacro:property name="calf_rotor_ixy" value="0.0"/>
-    <xacro:property name="calf_rotor_ixz" value="0.0"/>
-    <xacro:property name="calf_rotor_iyy" value="0.000111842"/>
-    <xacro:property name="calf_rotor_iyz" value="0.0"/>
-    <xacro:property name="calf_rotor_izz" value="0.000059647"/>
+    <xacro:property name="calf_mass" value="0.131"/>
+    <xacro:property name="calf_com_x" value="0.006286"/>
+    <xacro:property name="calf_com_y" value="0.001307"/>
+    <xacro:property name="calf_com_z" value="-0.122269"/>
+    <xacro:property name="calf_ixx" value="0.002939186297"/>
+    <xacro:property name="calf_ixy" value="0.000001440899"/>
+    <xacro:property name="calf_ixz" value="-0.000105359550"/>
+    <xacro:property name="calf_iyy" value="0.00295576935"/>
+    <xacro:property name="calf_iyz" value="-0.000024397752"/>
+    <xacro:property name="calf_izz" value="0.000030273372"/>
     <!-- foot -->
     <xacro:property name="foot_mass" value="0.06"/>

File: digital-twin-service/go1-base/catkin_ws/src/qre_go1/go1_description/xacro/leg.xacro (robot description, xacro)
@@ -2,18 +2,7 @@
 <robot xmlns:xacro="http://www.ros.org/wiki/xacro">
     <xacro:include filename="$(find go1_description)/xacro/transmission.xacro"/>
-    <xacro:macro name="leg" params="name mirror mirror_dae front_hind front_hind_dae">
+    <xacro:macro name="leg" params="name mirror mirror_dae front_hind front_hind_dae *origin">
         <joint name="${name}_hip_joint" type="revolute">
-            <xacro:if value="${(mirror_dae == False) and (front_hind_dae == True)}">
-                <origin rpy="0 0 0" xyz="${leg_offset_x} ${-leg_offset_y} 0"/>
-            </xacro:if>
-            <xacro:if value="${(mirror_dae == True) and (front_hind_dae == True)}">
-                <origin rpy="0 0 0" xyz="${leg_offset_x} ${leg_offset_y} 0"/>
-            </xacro:if>
-            <xacro:if value="${(mirror_dae == False) and (front_hind_dae == False)}">
-                <origin rpy="0 0 0" xyz="${-leg_offset_x} ${-leg_offset_y} 0"/>
-            </xacro:if>
-            <xacro:if value="${(mirror_dae == True) and (front_hind_dae == False)}">
-                <origin rpy="0 0 0" xyz="${-leg_offset_x} ${leg_offset_y} 0"/>
-            </xacro:if>
+            <xacro:insert_block name="origin"/>
             <parent link="trunk"/>
             <child link="${name}_hip"/>
@@ -21,25 +10,9 @@
             <dynamics damping="${damping}" friction="${friction}"/>
             <xacro:if value="${(mirror_dae == True)}">
-                <limit effort="${hip_torque_max}" velocity="${hip_velocity_max}" lower="${hip_position_min}" upper="${hip_position_max}"/>
+                <limit effort="${hip_torque_max}" velocity="${hip_velocity_max}" lower="${hip_min*PI/180.0}" upper="${hip_max*PI/180.0}"/>
             </xacro:if>
             <xacro:if value="${(mirror_dae == False)}">
-                <limit effort="${hip_torque_max}" velocity="${hip_velocity_max}" lower="${-hip_position_max}" upper="${-hip_position_min}"/>
+                <limit effort="${hip_torque_max}" velocity="${hip_velocity_max}" lower="${-hip_max*PI/180.0}" upper="${-hip_min*PI/180.0}"/>
             </xacro:if>
-        </joint>
-        <joint name="${name}_hip_rotor_joint" type="fixed">
-            <xacro:if value="${(mirror_dae == False) and (front_hind_dae == True)}">
-                <origin rpy="0 0 0" xyz="${hip_rotor_offset_x} ${-hip_rotor_offset_y} 0"/>
-            </xacro:if>
-            <xacro:if value="${(mirror_dae == True) and (front_hind_dae == True)}">
-                <origin rpy="0 0 0" xyz="${hip_rotor_offset_x} ${hip_rotor_offset_y} 0"/>
-            </xacro:if>
-            <xacro:if value="${(mirror_dae == False) and (front_hind_dae == False)}">
-                <origin rpy="0 0 0" xyz="${-hip_rotor_offset_x} ${-hip_rotor_offset_y} 0"/>
-            </xacro:if>
-            <xacro:if value="${(mirror_dae == True) and (front_hind_dae == False)}">
-                <origin rpy="0 0 0" xyz="${-hip_rotor_offset_x} ${hip_rotor_offset_y} 0"/>
-            </xacro:if>
-            <parent link="trunk"/>
-            <child link="${name}_hip_rotor"/>
         </joint>
         <link name="${name}_hip">
@@ -63,5 +36,5 @@
             </visual>
             <collision>
-                <origin rpy="${PI/2.0} 0 0" xyz="0 ${hip_offset*mirror} 0"/>
+                <origin rpy="${PI/2.0} 0 0" xyz="0 0 0"/>
                 <geometry>
                     <cylinder length="${hip_length}" radius="${hip_radius}"/>
@@ -77,26 +50,17 @@
             </inertial>
         </link>
-        <link name="${name}_hip_rotor">
-            <visual>
-                <origin rpy="0 ${PI/2.0} 0" xyz="0 0 0"/>
+        <joint name="${name}_hip_fixed" type="fixed">
+            <origin rpy="0 0 0" xyz="0 ${(hip_offset)*mirror} 0"/>
+            <parent link="${name}_hip"/>
+            <child link="${name}_thigh_shoulder"/>
+        </joint>
+        <!-- this link is only for collision -->
+        <link name="${name}_thigh_shoulder">
+            <collision>
+                <origin rpy="${PI/2.0} 0 0" xyz="0 0 0"/>
                 <geometry>
-                    <cylinder length="0.02" radius="0.035"/>
+                    <cylinder length="${thigh_shoulder_length}" radius="${thigh_shoulder_radius}"/>
                 </geometry>
-                <material name="green"/>
-            </visual>
-            <!-- <collision>
-                <origin rpy="0 ${PI/2.0} 0" xyz="0 0 0"/>
-                <geometry>
-                    <cylinder length="0.02" radius="0.035"/>
-                </geometry>
-            </collision> -->
-            <inertial>
-                <origin rpy="0 0 0" xyz="${hip_rotor_com_x} ${hip_rotor_com_y} ${hip_rotor_com_z}"/>
-                <mass value="${hip_rotor_mass}"/>
-                <inertia
-                    ixx="${hip_rotor_ixx}" ixy="${hip_rotor_ixy}" ixz="${hip_rotor_ixz}"
-                    iyy="${hip_rotor_iyy}" iyz="${hip_rotor_iyz}"
-                    izz="${hip_rotor_izz}"/>
-            </inertial>
+            </collision>
         </link>
         <joint name="${name}_thigh_joint" type="revolute">
@@ -106,10 +70,5 @@
             <axis xyz="0 1 0"/>
             <dynamics damping="${damping}" friction="${friction}"/>
-            <limit effort="${thigh_torque_max}" velocity="${thigh_velocity_max}" lower="${thigh_position_min}" upper="${thigh_position_max}"/>
-        </joint>
-        <joint name="${name}_thigh_rotor_joint" type="fixed">
-            <origin rpy="0 0 0" xyz="${thigh_rotor_offset_x} ${thigh_rotor_offset_y*mirror} 0"/>
-            <parent link="${name}_hip"/>
-            <child link="${name}_thigh_rotor"/>
+            <limit effort="${thigh_torque_max}" velocity="${thigh_velocity_max}" lower="${thigh_min*PI/180.0}" upper="${thigh_max*PI/180.0}"/>
         </joint>
         <link name="${name}_thigh">
@@ -141,27 +100,4 @@
             </inertial>
         </link>
-        <link name="${name}_thigh_rotor">
-            <visual>
-                <origin rpy="${PI/2.0} 0 0" xyz="0 0 0"/>
-                <geometry>
-                    <cylinder length="0.02" radius="0.035"/>
-                </geometry>
-                <material name="green"/>
-            </visual>
-            <!-- <collision>
-                <origin rpy="${PI/2.0} 0 0" xyz="0 0 0"/>
-                <geometry>
-                    <cylinder length="0.02" radius="0.035"/>
-                </geometry>
-            </collision> -->
-            <inertial>
-                <origin rpy="0 0 0" xyz="${thigh_rotor_com_x} ${thigh_rotor_com_y} ${thigh_rotor_com_z}"/>
-                <mass value="${thigh_rotor_mass}"/>
-                <inertia
-                    ixx="${thigh_rotor_ixx}" ixy="${thigh_rotor_ixy}" ixz="${thigh_rotor_ixz}"
-                    iyy="${thigh_rotor_iyy}" iyz="${thigh_rotor_iyz}"
-                    izz="${thigh_rotor_izz}"/>
-            </inertial>
-        </link>
         <joint name="${name}_calf_joint" type="revolute">
             <origin rpy="0 0 0" xyz="0 0 ${-thigh_length}"/>
@@ -170,10 +106,5 @@
             <axis xyz="0 1 0"/>
             <dynamics damping="${damping}" friction="${friction}"/>
-            <limit effort="${calf_torque_max}" velocity="${calf_velocity_max}" lower="${calf_position_min}" upper="${calf_position_max}"/>
-        </joint>
-        <joint name="${name}_calf_rotor_joint" type="fixed">
-            <origin rpy="0 0 0" xyz="${calf_rotor_offset_x} ${calf_rotor_offset_y*mirror} 0"/>
-            <parent link="${name}_thigh"/>
-            <child link="${name}_calf_rotor"/>
+            <limit effort="${calf_torque_max}" velocity="${calf_velocity_max}" lower="${calf_min*PI/180.0}" upper="${calf_max*PI/180.0}"/>
         </joint>
         <link name="${name}_calf">
@@ -198,27 +129,4 @@
                     iyy="${calf_iyy}" iyz="${calf_iyz}"
                     izz="${calf_izz}"/>
-            </inertial>
-        </link>
-        <link name="${name}_calf_rotor">
-            <visual>
-                <origin rpy="${PI/2.0} 0 0" xyz="0 0 0"/>
-                <geometry>
-                    <cylinder length="0.02" radius="0.035"/>
-                </geometry>
-                <material name="green"/>
-            </visual>
-            <!-- <collision>
-                <origin rpy="${PI/2.0} 0 0" xyz="0 0 0"/>
-                <geometry>
-                    <cylinder length="0.02" radius="0.035"/>
-                </geometry>
-            </collision> -->
-            <inertial>
-                <origin rpy="0 0 0" xyz="${calf_rotor_com_x} ${calf_rotor_com_y} ${calf_rotor_com_z}"/>
-                <mass value="${calf_rotor_mass}"/>
-                <inertia
-                    ixx="${calf_rotor_ixx}" ixy="${calf_rotor_ixy}" ixz="${calf_rotor_ixz}"
-                    iyy="${calf_rotor_iyy}" iyz="${calf_rotor_iyz}"
-                    izz="${calf_rotor_izz}"/>
             </inertial>
         </link>
