Commit message: a

File: digital-twin-service/go1-base/catkin_ws/src/qre_go1/go1_description/xacro/robot.xacro (robot description, xacro)
@@ -10,7 +10,8 @@
     <xacro:include filename="$(find go1_description)/xacro/ultraSound.xacro"/>
     <!-- <xacro:include filename="$(find go1_gazebo)/launch/stairs.urdf.xacro"/> -->
+    <xacro:include filename="$(find go1_description)/xacro/lidar.xacro"/>
     <!-- <xacro:stairs stairs="15" xpos="0" ypos="0" zpos="0" /> -->
-    <!-- Rotor related joint and link is only for demonstrate location. -->
-    <!-- Actually, the rotor will rotate and the joint is not fixed. Reduction ratio should be considered. -->
+    <!-- Rollover Protection mode will add an additional stick on the top, use "true" or "false" to switch it. -->
+    <xacro:property name="rolloverProtection" value="false"/>
     <!-- Debug mode will hung up the robot, use "true" or "false" to switch it. -->
     <xacro:if value="$(arg DEBUG)">
@@ -29,4 +30,25 @@
             </geometry>
         </visual>
+    </link>
+    <!-- Phidgets IMU mounted to the base frame -->
+    <joint name="phidgets_imu_joint" type="fixed">
+        <parent link="base"/>
+        <child link="phidgets_imu_link"/>
+        <!-- Set these to the IMU’s position/orientation relative to base -->
+        <origin xyz="0 0 0" rpy="0 0 0"/>
+    </joint>
+    <link name="phidgets_imu_link">
+        <inertial>
+            <mass value="0.001"/>
+            <origin xyz="0 0 0" rpy="0 0 0"/>
+            <inertia ixx="1e-4" ixy="0" ixz="0" iyy="1e-4" iyz="0" izz="1e-4"/>
+        </inertial>
+        <visual>
+            <geometry><box size="0.001 0.001 0.001"/></geometry>
+            <material name="black"/>
+        </visual>
+        <collision>
+            <geometry><box size="0.001 0.001 0.001"/></geometry>
+        </collision>
     </link>
     <joint name="floating_base" type="fixed">
@@ -58,4 +80,33 @@
         </inertial>
     </link>
+    <xacro:if value="${(rolloverProtection == 'true')}">
+        <joint name="stick_joint" type="fixed">
+            <parent link="trunk"/>
+            <child link="stick_link"/>
+            <origin rpy="0 0 0" xyz="${0.18} 0 ${stick_length/2.0+0.08}"/>
+        </joint>
+        <link name="stick_link">
+            <visual>
+                <geometry>
+                    <cylinder length="${stick_length}" radius="${stick_radius}"/>
+                </geometry>
+                <origin rpy="0 0 0" xyz="0 0 0"/>
+                <!-- <material name="white"/> -->
+            </visual>
+            <collision>
+                <geometry>
+                    <cylinder length="${stick_length}" radius="${stick_radius}"/>
+                </geometry>
+                <origin rpy="0 0 0" xyz="0 0 0"/>
+            </collision>
+            <inertial>
+                <mass value="${stick_mass}"/>
+                <inertia
+                    ixx="${stick_mass / 2.0 * (stick_radius*stick_radius)}" ixy="0.0" ixz="0.0"
+                    iyy="${stick_mass / 12.0 * (3*stick_radius*stick_radius + stick_length*stick_length)}" iyz="0.0"
+                    izz="${stick_mass / 12.0 * (3*stick_radius*stick_radius + stick_length*stick_length)}"/>
+            </inertial>
+        </link>
+    </xacro:if>
     <joint name="imu_joint" type="fixed">
         <parent link="trunk"/>
@@ -83,8 +134,16 @@
         </collision>
     </link>
-    <xacro:leg name="FR" mirror="-1" mirror_dae= "False" front_hind="1"  front_hind_dae="True"  />
-    <xacro:leg name="FL" mirror="1"  mirror_dae="True"   front_hind="1"  front_hind_dae="True"  />
-    <xacro:leg name="RR" mirror="-1" mirror_dae="False"  front_hind="-1" front_hind_dae="False" />
-    <xacro:leg name="RL" mirror="1"  mirror_dae="True"   front_hind="-1" front_hind_dae="False" />
+    <xacro:leg name="FR" mirror="-1" mirror_dae="False" front_hind="1" front_hind_dae="True">
+        <origin rpy="0 0 0" xyz="${leg_offset_x} ${-leg_offset_y} 0"/>
+    </xacro:leg>
+    <xacro:leg name="FL" mirror="1" mirror_dae="True" front_hind="1" front_hind_dae="True">
+        <origin rpy="0 0 0" xyz="${leg_offset_x} ${leg_offset_y} 0"/>
+    </xacro:leg>
+    <xacro:leg name="RR" mirror="-1" mirror_dae="False" front_hind="-1" front_hind_dae="False">
+        <origin rpy="0 0 0" xyz="${-leg_offset_x} ${-leg_offset_y} 0"/>
+    </xacro:leg>
+    <xacro:leg name="RL" mirror="1" mirror_dae="True" front_hind="-1" front_hind_dae="False">
+        <origin rpy="0 0 0" xyz="${-leg_offset_x} ${leg_offset_y} 0"/>
+    </xacro:leg>
     <xacro:depthCamera camID="1" name="face">
         <origin rpy="${PI} 0 0" xyz="0.2785 0.0125 0.0167"/>
@@ -125,3 +184,6 @@
         <origin rpy="0 0 0" xyz="0.2747 0.0 -0.0088"/>
     </xacro:ultraSound>
+    <xacro:lidar parent="trunk">
+        <origin rpy="0 0 0" xyz="0.05 0 0.08"/>
+    </xacro:lidar>
 </robot>

Commit message: cc

File: digital-twin-service/go1-base/catkin_ws/src/qre_go1/go1_description/xacro/robot.xacro (robot description, xacro)
@@ -14,4 +14,5 @@
     <!-- Rollover Protection mode will add an additional stick on the top, use "true" or "false" to switch it. -->
     <xacro:property name="rolloverProtection" value="false"/>
+    <xacro:property name="body_yaw_correction" value="3.141592653589793"/>  <!-- π -->
     <!-- Debug mode will hung up the robot, use "true" or "false" to switch it. -->
     <xacro:if value="$(arg DEBUG)">
@@ -25,5 +26,5 @@
     <link name="base">
         <visual>
-            <origin rpy="0 0 0" xyz="0 0 3.141592653589793"/>
+            <origin rpy="0 0 ${body_yaw_correction}" xyz="0 0 0"/>
             <geometry>
                 <box size="0.001 0.001 0.001"/>

Commit message: dd

File: digital-twin-service/go1-base/catkin_ws/src/qre_go1/go1_description/xacro/robot.xacro (robot description, xacro)
@@ -14,5 +14,4 @@
     <!-- Rollover Protection mode will add an additional stick on the top, use "true" or "false" to switch it. -->
     <xacro:property name="rolloverProtection" value="false"/>
-    <xacro:property name="body_yaw_correction" value="3.141592653589793"/>  <!-- π -->
     <!-- Debug mode will hung up the robot, use "true" or "false" to switch it. -->
     <xacro:if value="$(arg DEBUG)">
@@ -26,5 +25,5 @@
     <link name="base">
         <visual>
-            <origin rpy="0 0 ${body_yaw_correction}" xyz="0 0 0"/>
+            <origin rpy="0 0 0" xyz="0 0 0"/>
             <geometry>
                 <box size="0.001 0.001 0.001"/>
